Commit message: 2.6

File: ServoControl/arm.urdf (robot description, URDF)
Before this commit: robot chess_arm, 7 links, 6 joints
Links:
- removed link tool_tip
- added link grasp_target
- link base_link: geometry 
Joints:
- removed joint s5_gripper
- added joint gripper_tip_joint: type fixed, parent link_s5, child grasp_target, origin xyz=0 0 0 rpy=0 0 0
- joint s1_pitch: origin xyz=0.1 0.1 0.3 rpy=0 0 0 -> xyz=0.015 0.01 0.025 rpy=0 0 0
- joint s2_pitch: origin xyz=0 0 0.15 rpy=0 0 0 -> xyz=0 0 0.105 rpy=0 1.5708 0
- joint s3_pitch: origin xyz=0 0 0.104 rpy=0 0 0 -> xyz=0.025 0 -0.05 rpy=0 1.5708 0
- joint s4_roll: limit lower=-1.57 upper=1.57 effort=1.0 velocity=1.0 -> lower=-3.14 upper=3.14 effort=1.0 velocity=1.0; origin xyz=0 0.1 0 rpy=0 0 0 -> xyz=0.02 0 -0.10 rpy=0 0 0
